File: hat_rspi_7segdisplay.sch (EAGLE design)
At the start: 0 parts

Commit message: Add files via upload
Parts:
- added IC1: (no value), max6958:MAX6958
- added X1: RASPI_BOARD_AB_E0, raspberrypi_bastelstube_v13:RASPI_BOARD_AB_E0
Changed lines of the file:
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@@
 <layer number="48" name="Document" color="7" fill="1" visible="no" active="no"/>
 <layer number="49" name="Reference" color="7" fill="1" visible="no" active="no"/>
+<layer number="50" name="dxf" color="7" fill="1" visible="no" active="no"/>
 <layer number="51" name="tDocu" color="7" fill="1" visible="no" active="no"/>
 <layer number="52" name="bDocu" color="7" fill="1" visible="no" active="no"/>
@@
 <layer number="97" name="Info" color="7" fill="1" visible="yes" active="yes"/>
 <layer number="98" name="Guide" color="6" fill="1" visible="yes" active="yes"/>
+<layer number="250" name="Descript" color="3" fill="1" visible="no" active="no"/>
+<layer number="251" name="SMDround" color="12" fill="11" visible="no" active="no"/>
 </layers>
 <schematic xreflabel="%F%N/%S.%C%R" xrefpart="/%S.%C%R">
@@
 <part name="FRAME1" library="frames" library_urn="urn:adsk.eagle:library:229" deviceset="A3L-LOC" device=""/>
 <part name="FRAME2" library="frames" library_urn="urn:adsk.eagle:library:229" deviceset="A3L-LOC" device=""/>
+<part name="IC1" library="max6958" deviceset="MAX6958" device=""/>
+<part name="X1" library="raspberrypi_bastelstube_v13" deviceset="RASPI_BOARD_AB" device="_E0"/>
 </parts>
 <sheets>
@@
 <attribute name="SHEET" x="357.505" y="5.08" size="2.54" layer="94"/>
 </instance>
+<instance part="IC1" gate="G$1" x="187.96" y="142.24" smashed="yes">
+<attribute name="NAME" x="183.1975" y="160.02" size="1.27" layer="95" rot="R180"/>
+<attribute name="VALUE" x="176.8475" y="123.5075" size="1.27" layer="96"/>
+</instance>
+<instance part="X1" gate="G$1" x="119.38" y="144.78" smashed="yes"/>
 </instances>
 <busses>
