File: hat_rspi_7segdisplay.sch (EAGLE design)
At the start: 0 parts

Commit message: adding some resistors
Parts:
- added IC1: (no value), max6958:MAX6958
- added R1, R2, R3, R4, R5, R6, R7, R8: (no value), rcl:R-EU_0204/5
- added U1: 5641AH, hat_rpi_7segdisplay:5641AH
- added X1: RASPI_BOARD_AB_E0, raspberrypi_bastelstube_v13:RASPI_BOARD_AB_E0
Connections:
- new net N$1: IC1.GND, X1.GND
- new net N$2: X1.SCL
- new net N$3: IC1.SCL
- new net N$4: IC1.SDA, X1.SDA
- new net N$5: R3.1, U1.A8
Changed lines of the file:
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@@
 <setting verticaltext="up"/>
 </settings>
-<grid distance="0.1" unitdist="inch" unit="inch" style="lines" multiple="1" display="no" altdistance="0.01" altunitdist="inch" altunit="inch"/>
+<grid distance="1" unitdist="mm" unit="mm" style="lines" multiple="1" display="no" altdistance="0.01" altunitdist="inch" altunit="inch"/>
 <layers>
 <layer number="1" name="Top" color="4" fill="1" visible="no" active="no"/>
@@
 <layer number="48" name="Document" color="7" fill="1" visible="no" active="no"/>
 <layer number="49" name="Reference" color="7" fill="1" visible="no" active="no"/>
+<layer number="50" name="dxf" color="7" fill="1" visible="no" active="no"/>
 <layer number="51" name="tDocu" color="7" fill="1" visible="no" active="no"/>
 <layer number="52" name="bDocu" color="7" fill="1" visible="no" active="no"/>
@@
 <layer number="97" name="Info" color="7" fill="1" visible="yes" active="yes"/>
 <layer number="98" name="Guide" color="6" fill="1" visible="yes" active="yes"/>
+<layer number="250" name="Descript" color="3" fill="1" visible="no" active="no"/>
+<layer number="251" name="SMDround" color="12" fill="11" visible="no" active="no"/>
 </layers>
 <schematic xreflabel="%F%N/%S.%C%R" xrefpart="/%S.%C%R">
@@
 <parts>
 <part name="FRAME1" library="frames" library_urn="urn:adsk.eagle:library:229" deviceset="A3L-LOC" device=""/>
-<part name="FRAME2" library="frames" library_urn="urn:adsk.eagle:library:229" deviceset="A3L-LOC" device=""/>
+<part name="IC1" library="max6958" deviceset="MAX6958" device=""/>
+<part name="X1" library="raspberrypi_bastelstube_v13" deviceset="RASPI_BOARD_AB" device="_E0"/>
+<part name="U1" library="hat_rpi_7segdisplay" deviceset="5641AH" device=""/>
+<part name="R1" library="rcl" library_urn="urn:adsk.eagle:library:334" deviceset="R-EU_" device="0204/5" package3d_urn="urn:adsk.eagle:package:23488/1"/>
+<part name="R2" library="rcl" library_urn="urn:adsk.eagle:library:334" deviceset="R-EU_" device="0204/5" package3d_urn="urn:adsk.eagle:package:23488/1"/>
+<part name="R3" library="rcl" library_urn="urn:adsk.eagle:library:334" deviceset="R-EU_" device="0204/5" package3d_urn="urn:adsk.eagle:package:23488/1"/>
+<part name="R4" library="rcl" library_urn="urn:adsk.eagle:library:334" deviceset="R-EU_" device="0204/5" package3d_urn="urn:adsk.eagle:package:23488/1"/>
+<part name="R5" library="rcl" library_urn="urn:adsk.eagle:library:334" deviceset="R-EU_" device="0204/5" package3d_urn="urn:adsk.eagle:package:23488/1"/>
+<part name="R6" library="rcl" library_urn="urn:adsk.eagle:library:334" deviceset="R-EU_" device="0204/5" package3d_urn="urn:adsk.eagle:package:23488/1"/>
+<part name="R7" library="rcl" library_urn="urn:adsk.eagle:library:334" deviceset="R-EU_" device="0204/5" package3d_urn="urn:adsk.eagle:package:23488/1"/>
+<part name="R8" library="rcl" library_urn="urn:adsk.eagle:library:334" deviceset="R-EU_" device="0204/5" package3d_urn="urn:adsk.eagle:package:23488/1"/>
 </parts>
 <sheets>
@@
 </plain>
 <instances>
-<instance part="FRAME1" gate="G$1" x="0" y="0" smashed="yes">
-<attribute name="DRAWING_NAME" x="344.17" y="15.24" size="2.54" layer="94"/>
-<attribute name="LAST_DATE_TIME" x="344.17" y="10.16" size="2.286" layer="94"/>
-<attribute name="SHEET" x="357.505" y="5.08" size="2.54" layer="94"/>
-</instance>
-<instance part="FRAME2" gate="G$1" x="0" y="0" smashed="yes">
-<attribute name="DRAWING_NAME" x="344.17" y="15.24" size="2.54" layer="94"/>
-<attribute name="LAST_DATE_TIME" x="344.17" y="10.16" size="2.286" layer="94"/>
-<attribute name="SHEET" x="357.505" y="5.08" size="2.54" layer="94"/>
+<instance part="FRAME1" gate="G$1" x="-102" y="5" smashed="yes">
+<attribute name="DRAWING_NAME" x="242.17" y="20.24" size="2.54" layer="94"/>
+<attribute name="LAST_DATE_TIME" x="242.17" y="15.16" size="2.286" layer="94"/>
+<attribute name="SHEET" x="255.505" y="10.08" size="2.54" layer="94"/>
+</instance>
+<instance part="IC1" gate="G$1" x="88.9" y="132.08" smashed="yes">
+<attribute name="NAME" x="84.1375" y="149.86" size="1.27" layer="95" rot="R180"/>
+<attribute name="VALUE" x="77.7875" y="113.3475" size="1.27" layer="96"/>
+</instance>
+<instance part="X1" gate="G$1" x="22.86" y="134.62" smashed="yes"/>
+<instance part="U1" gate="G$1" x="165.968" y="127.884" smashed="yes" rot="R270">
+<attribute name="NAME" x="177.398" y="132.964" size="1.27" layer="95" rot="R270"/>
+<attribute name="VALUE" x="150.728" y="132.964" size="1.27" layer="96" rot="R270"/>
+</instance>
+<instance part="R1" gate="G$1" x="163.423" y="107.304" smashed="yes" rot="R90">
+<attribute name="NAME" x="161.9244" y="103.494" size="1.778" layer="95" rot="R90"/>
+<attribute name="VALUE" x="166.725" y="103.494" size="1.778" layer="96" rot="R90"/>
+</instance>
+<instance part="R2" gate="G$1" x="165.645" y="101.696" smashed="yes" rot="R270">
+<attribute name="NAME" x="167.1436" y="105.506" size="1.778" layer="95" rot="R270"/>
+<attribute name="VALUE" x="162.343" y="105.506" size="1.778" layer="96" rot="R270"/>
+</instance>
+<instance part="R3" gate="G$1" x="156.082" y="107.833" smashed="yes" rot="R270">
+<attribute name="NAME" x="157.5806" y="111.643" size="1.778" layer="95" rot="R270"/>
+<attribute name="VALUE" x="152.78" y="111.643" size="1.778" layer="96" rot="R270"/>
+</instance>
+<instance part="R4" gate="G$1" x="168.435" y="107.923" smashed="yes" rot="R270">
+<attribute name="NAME" x="169.9336" y="111.733" size="1.778" layer="95" rot="R270"/>
+<attribute name="VALUE" x="165.133" y="111.733" size="1.778" layer="96" rot="R270"/>
+</instance>
+<instance part="R5" gate="G$1" x="158.428" y="99.923" smashed="yes" rot="R270">
+<attribute name="NAME" x="159.9266" y="103.733" size="1.778" layer="95" rot="R270"/>
+<attribute name="VALUE" x="155.126" y="103.733" size="1.778" layer="96" rot="R270"/>
+</instance>
+<instance part="R6" gate="G$1" x="170.336" y="99.077" smashed="yes" rot="R90">
+<attribute name="NAME" x="168.8374" y="95.267" size="1.778" layer="95" rot="R90"/>
+<attribute name="VALUE" x="173.638" y="95.267" size="1.778" layer="96" rot="R90"/>
+</instance>
+<instance part="R7" gate="G$1" x="160.779" y="93.166" smashed="yes" rot="R270">
+<attribute name="NAME" x="162.2776" y="96.976" size="1.778" layer="95" rot="R270"/>
+<attribute name="VALUE" x="157.477" y="96.976" size="1.778" layer="96" rot="R270"/>
+</instance>
+<instance part="R8" gate="G$1" x="173.258" y="93.287" smashed="yes" rot="R270">
+<attribute name="NAME" x="174.7566" y="97.097" size="1.778" layer="95" rot="R270"/>
+<attribute name="VALUE" x="169.956" y="97.097" size="1.778" layer="96" rot="R270"/>
 </instance>
 </instances>
@@
 </busses>
 <nets>
+<net name="N$1" class="0">
+<segment>
+<pinref part="X1" gate="G$1" pin="GND"/>
+<wire x1="22.86" y1="109.22" x2="22.86" y2="104.14" width="0.1524" layer="91"/>
+<pinref part="IC1" gate="G$1" pin="GND"/>
+<wire x1="22.86" y1="104.14" x2="71.12" y2="104.14" width="0.1524" layer="91"/>
+<wire x1="71.12" y1="104.14" x2="71.12" y2="119.38" width="0.1524" layer="91"/>
+</segment>
+</net>
+<net name="N$2" class="0">
+<segment>
+<pinref part="X1" gate="G$1" pin="SCL"/>
+<wire x1="7.62" y1="119.38" x2="4.248" y2="119.38" width="0.1524" layer="91"/>
+<wire x1="4.248" y1="119.38" x2="4.248" y2="86.083" width="0.1524" layer="91"/>
+<wire x1="4.248" y1="86.083" x2="64.208" y2="86.083" width="0.1524" layer="91"/>
+<wire x1="64.208" y1="86.083" x2="64.26" y2="136.93" width="0.1524" layer="91"/>
+</segment>
+</net>
+<net name="N$3" class="0">
+<segment>
+<pinref part="IC1" gate="G$1" pin="SCL"/>
+<wire x1="76.2" y1="136.956" x2="76.2" y2="137.16" width="0.1524" layer="91"/>
+<wire x1="64.256" y1="136.919" x2="64.264" y2="137.152" width="0.1524" layer="91"/>
+<wire x1="64.264" y1="137.152" x2="76.169" y2="137.143" width="0.1524" layer="91"/>
+<wire x1="76.169" y1="137.143" x2="76.2" y2="137.16" width="0.1524" layer="91"/>
+<junction x="76.2" y="137.16"/>
+</segment>
+</net>
+<net name="N$4" class="0">
+<segment>
+<pinref part="X1" gate="G$1" pin="SDA"/>
+<wire x1="7.62" y1="116.84" x2="5.258" y2="116.84" width="0.1524" layer="91"/>
+<wire x1="5.258" y1="116.84" x2="5.258" y2="87.298" width="0.1524" layer="91"/>
+<wire x1="5.258" y1="87.298" x2="62.491" y2="87.298" width="0.1524" layer="91"/>
+<pinref part="IC1" gate="G$1" pin="SDA"/>
+<wire x1="62.491" y1="87.298" x2="62.491" y2="139.7" width="0.1524" layer="91"/>
+<wire x1="62.491" y1="139.7" x2="76.2" y2="139.7" width="0.1524" layer="91"/>
+</segment>
+</net>
+<net name="N$5" class="0">
+<segment>
+<pinref part="U1" gate="G$1" pin="A8"/>
+<pinref part="R3" gate="G$1" pin="1"/>
+<wire x1="155.808" y1="115.184" x2="156.082" y2="115.184" width="0.1524" layer="91"/>
+<wire x1="156.082" y1="115.184" x2="156.082" y2="112.913" width="0.1524" layer="91"/>
+</segment>
+</net>
 </nets>
 </sheet>
@@
 will not be understood (or retained) with this version.
 </note>
+<note version="8.3" severity="warning">
+Since Version 8.3, EAGLE supports the association of 3D packages
+with devices in libraries, schematics, and board files. Those 3D
+packages will not be understood (or retained) with this version.
+</note>
+<note version="8.4" severity="warning">
+Since Version 8.4, EAGLE supports properties for SPICE simulation.
+Probes in schematics and SPICE mapping objects found in parts and library devices
+will not be understood with this version. Update EAGLE to the latest version
+for full support of SPICE simulation.
+</note>
 </compatibility>
