File: hat_raspi_7segdis.sch (EAGLE design)
At the start: 2 parts, among them X1 RASPI_BOARD_AB_E0

Commit message: first draft to be sent
Parts:
- added R1, R2: 39kΩ, Resistor:R_AXIAL-7.2MM-PITCH
- added R3, R4, R5: 10Ω, Resistor:R_AXIAL-7.2MM-PITCH
- added R6: 100Ω, Resistor:R_AXIAL-7.2MM-PITCH
- added U1: 5641AH, hat_rpi_7segdisplay:5641AH
- IC1: device max6958:MAX6958 -> hat_rpi_7segdisplay:MAX6958
- X1: value RASPI_BOARD_AB_E0 -> RASPI_BOARD_AB_E2P; device raspberrypi_bastelstube_v13:RASPI_BOARD_AB_E0 -> hat_rpi_7segdisplay:RASPI_BOARD_AB_E2P
Connections:
- new net N$1: R4.2, U1.K4
- new net N$10: IC1.SEG2, R1.1
- new net N$11: R2.1, U1.A1, U1.A2, U1.A3, U1.A4
- new net N$12: R1.2, U1.A5, U1.A6, U1.A7, U1.A8
- new net N$13: IC1.SCL, X1.SCL
- new net N$14: IC1.SDA, X1.SDA
- new net N$15: IC1.VCC, X1.5V0
- new net N$2: R3.1, U1.K3
- new net N$3: R5.2, U1.K2
- new net N$4: R6.2, U1.K1
- new net N$5: R3.2, R4.1, R5.1, R6.1, X1.GND
- new net N$9: IC1.SEG1, R2.2
Other:
- moved on the sheet: IC1
